File: hardware/LINBoard/LINBoard.kicad_sch (KiCad schematic)
At the start: 10 parts, among them J1 Conn_01x02_Pin, SW1 SW_SPDT, U1 TLIN2029ADRQ1

Commit message: Updated step files for all boards, footprints for LINBoard.
Parts:
- C1, C2: footprint PCM_Capacitor_SMD_AKL:C_0805_2012Metric -> Capacitor_SMD:C_0805_2012Metric
- D1: footprint PCM_Diode_SMD_AKL:D_SOD-123 -> Diode_SMD:D_SOD-123
- J2: value (none) -> ~
- R1, R2, R3: footprint PCM_Resistor_SMD_AKL:R_0805_2012Metric -> Resistor_SMD:R_0805_2012Metric
Changed lines of the file:
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@@
 			)
 		)
-		(property "Footprint" "PCM_Capacitor_SMD_AKL:C_0805_2012Metric"
+		(property "Footprint" "Capacitor_SMD:C_0805_2012Metric"
 			(at 84.7852 48.26 0)
 			(effects
@@
 			)
 		)
-		(property "Footprint" "PCM_Resistor_SMD_AKL:R_0805_2012Metric"
+		(property "Footprint" "Resistor_SMD:R_0805_2012Metric"
 			(at 35.56 40.64 0)
 			(effects
@@
 			)
 		)
-		(property "Footprint" "PCM_Resistor_SMD_AKL:R_0805_2012Metric"
+		(property "Footprint" "Resistor_SMD:R_0805_2012Metric"
 			(at 77.47 19.05 0)
 			(effects
@@
 			)
 		)
-		(property "Footprint" "PCM_Capacitor_SMD_AKL:C_0805_2012Metric"
+		(property "Footprint" "Capacitor_SMD:C_0805_2012Metric"
 			(at 31.75 18.0848 0)
 			(effects
@@
 			)
 		)
-		(property "Footprint" "PCM_Diode_SMD_AKL:D_SOD-123"
+		(property "Footprint" "Diode_SMD:D_SOD-123"
 			(at 55.88 19.05 0)
 			(effects
@@
 			)
 		)
-		(property "Footprint" "PCM_Resistor_SMD_AKL:R_0805_2012Metric"
+		(property "Footprint" "Resistor_SMD:R_0805_2012Metric"
 			(at 25.4 40.64 0)
 			(effects
@@
 			)
 		)
-		(property "Value" ""
+		(property "Value" "~"
 			(at 17.145 31.75 0)
 			(effects

Commit message: Updated LINboard to kicad v10. Added pcis.
Parts:
- J2: value ~ -> (none)
