File: hardware/ETHBoard/ETHBoard.kicad_pcb (KiCad board)
At the start: 2 copper layers, 25.1 x 12.2 mm, 34 parts, among them J1 Conn_02x04_Odd_Even, J2 Conn_01x02_Pin, U1 LAN8651B1-E_LMX, Y1 X322525MOB4SI

Commit message: ETHBoard: Slightly moved bottom side components.
Parts:
- moved R5 0.85 mm to (95.1, 61.2)
- moved R6 0.85 mm to (95.1, 52.6)
- moved C18 0.54 mm to (91.8, 59.8)
- moved C19 0.54 mm to (91.8, 54.0)
- moved R7 0.25 mm to (89.7, 54.6)
- moved R8 0.25 mm to (89.7, 59.2)
- moved R1 0.16 mm to (84.0, 62.0)
- moved R2 0.15 mm to (80.3, 52.5)
- moved C1 0.10 mm to (83.4, 60.7)
Routing:
- net /T1S_d-: track 9.89 -> 10.8 mm
- net /T1S_d+: track 9.89 -> 10.8 mm
- net GND: vias 30 -> 29
